File: card_pcb/card_pcb.sch (KiCad schematic (older format))
At the start: 41 parts

Commit message: a trim off the top
Parts:
- G5: footprint mylogos:fungi_2 -> mylogos:fungi_2_trim
Changed lines of the file:
@@
 EESchema Schematic File Version 4
+LIBS:card_pcb-cache
 EELAYER 26 0
 EELAYER END
@@
 F 0 "G5" H 7900 3642 60  0001 C CNN
 F 1 "LOGO" H 7900 5708 60  0001 C CNN
-F 2 "mylogos:fungi_2" H 7900 4675 50  0001 C CNN
+F 2 "mylogos:fungi_2_trim" H 7900 4675 50  0001 C CNN
 F 3 "" H 7900 4675 50  0001 C CNN
 	1    7900 4675
